Commit message: urdf fixed,gazebo runs expectedly for now

File: mybot/urdf/mybot.urdf_actual.xacro (robot description, xacro)
@@ -12,73 +12,10 @@
     <color rgba="1.0 0.5 0.5 1.0" />
   </material>
-  <material name="grey">
-    <color rgba="0.5 0.5 0.5 1.0"/>
-  </material>
-  <!-- _________________________________ -->
-  <link name="world"/>
-  <joint name="fixed_world" type="fixed">
-    <parent link="world"/>
-    <child link="base_plane"/>
-  </joint>
-  <link name="base_bar">
-    <!--inertial>
-            <origin rpy="0 0 0" xyz="0 0 0" />
-            <mass value="0.392347184025621" />
-            <inertia ixx="0.0" ixy="0" ixz="0" iyy="0" iyz="0" izz="0" />
-        </inertial-->
-    <visual>
-      <origin xyz="0.0 0.0 0.05" rpy="0.0 0.0 0.0"/>
-      <geometry>
-        <box size="0.01 0.01 0.1"/>
-      </geometry>
-      <material name="pink"/>
-    </visual>
-    <collision>
-      <origin xyz="0.0 0.0 0.05" rpy="0.0 0.0 0.0"/>
-      <geometry>
-        <box size="0.01 0.01 0.1"/>
-      </geometry>
-    </collision>
-  </link>
-  <joint name="base_bar__base_plane" type="fixed">
-    <origin xyz="0.0 0.0 0.0" rpy="0.0 0.0 0.0"/>
-    <parent link="base_plane"/>
-    <child link="base_bar"/>
-    <axis xyz="0.0 0.0 0.0"/>
-    <limit lower="0.0" upper="0.0" effort="1000.0" velocity="50.0"/>
-  </joint>
-  <joint name="base_plane__ArmBase" type="fixed">
-        <origin rpy="0.0 0.0 0.0" xyz="0.0 0.0 0.5" />
-        <parent link="base_bar" />
-        <child link="base" />
-        <axis xyz="0.0 0.0 0.0" />
-        <limit lower="0.0" upper="0.0" effort="1000.0" velocity="50.0"/>
-    </joint>
-  <link name="base_plane">
-    <!--inertial>
-            <origin rpy="0 0 0" xyz="0 0 0" />
-            <mass value="0.392347184025621" />
-            <inertia ixx="0.0" ixy="0" ixz="0" iyy="0" iyz="0" izz="0" />
-        </inertial-->
-    <visual name="">
-      <origin xyz="0.0 0.0 0.01" rpy="0.0 0.0 0.0"/>
-      <geometry>
-        <box size="1.5 1.5 0.02"/>
-      </geometry>
-      <material name="grey"/>
-    </visual>
-    <collision>
-      <origin xyz="0.0 0.0 0.01" rpy="0.0 0.0 0.0"/>
-      <geometry>
-        <box size="1.5 1.5 0.02"/>
-      </geometry>
-    </collision>
-  </link>
-  <!-- _________________________________ -->
   <link name="base">
     <inertial>
       <origin rpy="0 0 0" xyz="-0.0024988 0.00012827 0.034299" />
       <mass value="1.2649" />
-      <inertia ixx="0.002533" ixy="-7.2003E-06" ixz="8.109E-05" iyy="0.0023931" iyz="-4.1626E-06" izz="0.0041505" />
+      <inertia ixx="0.002533" ixy="-7.2003E-06" ixz="8.109E-05" iyy="0.0023931" iyz="-4.1626E-06"
+        izz="0.0041505" />
     </inertial>
     <visual>
@@ -102,5 +39,6 @@
       <origin rpy="0 0 0" xyz="-0.00087897 0.0045493 0.030537" />
       <mass value="0.69097" />
-      <inertia ixx="0.00068689" ixy="3.5558E-06" ixz="1.3086E-05" iyy="0.00097033" iyz="-1.1454E-05" izz="0.0012375" />
+      <inertia ixx="0.00068689" ixy="3.5558E-06" ixz="1.3086E-05" iyy="0.00097033" iyz="-1.1454E-05"
+        izz="0.0012375" />
     </inertial>
     <visual>
@@ -131,5 +69,6 @@
       <origin rpy="0 0 0" xyz="-0.043702 -0.0089462 0.088598" />
       <mass value="0.50956" />
-      <inertia ixx="0.0022353" ixy="5.0525E-05" ixz="0.00097691" iyy="0.0027432" iyz="-0.00010402" izz="0.00069497" />
+      <inertia ixx="0.0022353" ixy="5.0525E-05" ixz="0.00097691" iyy="0.0027432" iyz="-0.00010402"
+        izz="0.00069497" />
     </inertial>
     <visual>
@@ -161,5 +100,6 @@
       <origin rpy="0 0 0" xyz="0.10764 0.020329 0.0017657" />
       <mass value="0.31089" />
-      <inertia ixx="9.4078E-05" ixy="1.6899E-07" ixz="-2.6416E-05" iyy="0.0017716" iyz="2.7724E-09" izz="0.001704" />
+      <inertia ixx="9.4078E-05" ixy="1.6899E-07" ixz="-2.6416E-05" iyy="0.0017716" iyz="2.7724E-09"
+        izz="0.001704" />
     </inertial>
     <visual>
@@ -192,5 +132,6 @@
       <origin rpy="0 0 0" xyz="0.10059 -0.0011654 -0.0095762" />
       <mass value="0.21582" />
-      <inertia ixx="5.0445E-05" ixy="-1.9198E-05" ixz="3.0188E-05" iyy="0.00021644" iyz="2.8871E-06" izz="0.00023311" />
+      <inertia ixx="5.0445E-05" ixy="-1.9198E-05" ixz="3.0188E-05" iyy="0.00021644" iyz="2.8871E-06"
+        izz="0.00023311" />
     </inertial>
     <visual>

File: prochesta_arm/urdf/prochesta_arm.urdf.xacro (robot description, xacro)
@@ -26,26 +26,28 @@
         <color rgba="0.0 1.0 0.5 1.0" />
     </material>
+    <!-- _________________________________ -->
     <link name="world"/>
     <joint name="fixed_world" type="fixed">
+        <origin xyz="0.0 0.0 0.0" rpy="0.0 0.0 0.0"/>
         <parent link="world"/>
         <child link="base_plane"/>
     </joint>
-    <link name="base_bar">
-        <!--inertial>
+    <link name="base_plane">
+        <inertial>
             <origin rpy="0 0 0" xyz="0 0 0" />
             <mass value="0.392347184025621" />
             <inertia ixx="0.0" ixy="0" ixz="0" iyy="0" iyz="0" izz="0" />
-        </inertial-->
-        <visual>
-            <origin xyz="0.0 0.0 0.05" rpy="0.0 0.0 0.0"/>
-            <geometry>
-                <box size="0.01 0.01 0.1"/>
+        </inertial>
+        <visual name="">
+            <origin xyz="0.0 0.0 0.01" rpy="0.0 0.0 0.0"/>
+            <geometry>
+                <box size="1.5 1.5 0.02"/>
             </geometry>
             <material name="grey"/>
         </visual>
         <collision>
-            <origin xyz="0.0 0.0 0.05" rpy="0.0 0.0 0.0"/>
-            <geometry>
-                <box size="0.01 0.01 0.1"/>
+            <origin xyz="0.0 0.0 0.01" rpy="0.0 0.0 0.0"/>
+            <geometry>
+                <box size="1.5 1.5 0.02"/>
             </geometry>
         </collision>
@@ -65,24 +67,25 @@
         <limit lower="0.0" upper="0.0" effort="1000.0" velocity="50.0"/>
     </joint>
-    <link name="base_plane">
-        <!--inertial>
+    <link name="base_bar">
+        <inertial>
             <origin rpy="0 0 0" xyz="0 0 0" />
             <mass value="0.392347184025621" />
             <inertia ixx="0.0" ixy="0" ixz="0" iyy="0" iyz="0" izz="0" />
-        </inertial-->
-        <visual name="">
-            <origin xyz="0.0 0.0 0.01" rpy="0.0 0.0 0.0"/>
-            <geometry>
-                <box size="1.5 1.5 0.02"/>
+        </inertial>
+        <visual>
+            <origin xyz="0.0 0.0 0.05" rpy="0.0 0.0 0.0"/>
+            <geometry>
+                <box size="0.01 0.01 0.1"/>
             </geometry>
             <material name="grey"/>
         </visual>
         <collision>
-            <origin xyz="0.0 0.0 0.01" rpy="0.0 0.0 0.0"/>
-            <geometry>
-                <box size="1.5 1.5 0.02"/>
-            </geometry>
-        </collision>
-    </link>
+            <origin xyz="0.0 0.0 0.05" rpy="0.0 0.0 0.0"/>
+            <geometry>
+                <box size="0.01 0.01 0.1"/>
+            </geometry>
+        </collision>
+    </link>
+    <!-- _________________________________ -->
     <link name="ArmBase">
         <inertial>
@@ -410,24 +413,4 @@
         </joint>
         <actuator name="Joint_RightClaw_motor">
-            <hardwareInterface>hardware_interface/PositionJointInterface</hardwareInterface>
-            <mechanicalReduction>1</mechanicalReduction>
-        </actuator>
-    </transmission>
-    <transmission name="trans_base_plane__ArmBase">
-        <type>transmission_interface/SimpleTransmission</type>
-        <joint name="base_plane__ArmBase">
-            <hardwareInterface>hardware_interface/PositionJointInterface</hardwareInterface>
-        </joint>
-        <actuator name="base_plane__ArmBase_motor">
-            <hardwareInterface>hardware_interface/PositionJointInterface</hardwareInterface>
-            <mechanicalReduction>1</mechanicalReduction>
-        </actuator>
-    </transmission>
-    <transmission name="trans_base_bar__base_plane">
-        <type>transmission_interface/SimpleTransmission</type>
-        <joint name="base_bar__base_plane">
-            <hardwareInterface>hardware_interface/PositionJointInterface</hardwareInterface>
-        </joint>
-        <actuator name="base_bar__base_plane_motor">
             <hardwareInterface>hardware_interface/PositionJointInterface</hardwareInterface>
             <mechanicalReduction>1</mechanicalReduction>
