Commit message: added world fixed joint

File: prochesta_arm/urdf/prochesta_arm.urdf.xacro (robot description, xacro)
@@ -26,4 +26,9 @@
         <color rgba="0.0 1.0 0.5 1.0" />
     </material>
+    <link name="world"/>
+    <joint name="fixed_world" type="fixed">
+        <parent link="world"/>
+        <child link="base_plane"/>
+    </joint>
     <link name="base_bar">
         <!--inertial>
@@ -58,5 +63,5 @@
         <child link="base_bar"/>
         <axis xyz="0.0 0.0 0.0"/>
-        <limit lower="0.0" upper="0.0" effort="0.0" velocity="0.0"/>
+        <limit lower="0.0" upper="0.0" effort="1000.0" velocity="50.0"/>
     </joint>
     <link name="base_plane">

Commit message: prochesta_motion added.

File: prochesta_arm/urdf/prochesta_arm.urdf.xacro (robot description, xacro)
@@ -340,8 +340,8 @@
         <type>transmission_interface/SimpleTransmission</type>
         <joint name="ArmBase__BaseShaft">
-            <hardwareInterface>hardware_interface/PositionJointInterface</hardwareInterface>
+            <hardwareInterface>hardware_interface/VelocityJointInterface</hardwareInterface>
         </joint>
         <actuator name="ArmBase__BaseShaft_motor">
-            <hardwareInterface>hardware_interface/PositionJointInterface</hardwareInterface>
+            <hardwareInterface>hardware_interface/VelocityJointInterface</hardwareInterface>
             <mechanicalReduction>1</mechanicalReduction>
         </actuator>
@@ -350,8 +350,8 @@
         <type>transmission_interface/SimpleTransmission</type>
         <joint name="BaseShaft__Shoulder">
-            <hardwareInterface>hardware_interface/PositionJointInterface</hardwareInterface>
+            <hardwareInterface>hardware_interface/VelocityJointInterface</hardwareInterface>
         </joint>
         <actuator name="BaseShaft__Shoulder_motor">
-            <hardwareInterface>hardware_interface/PositionJointInterface</hardwareInterface>
+            <hardwareInterface>hardware_interface/VelocityJointInterface</hardwareInterface>
             <mechanicalReduction>1</mechanicalReduction>
         </actuator>
@@ -360,8 +360,8 @@
         <type>transmission_interface/SimpleTransmission</type>
         <joint name="Shoulder__Elbow">
-            <hardwareInterface>hardware_interface/PositionJointInterface</hardwareInterface>
+            <hardwareInterface>hardware_interface/VelocityJointInterface</hardwareInterface>
         </joint>
         <actuator name="Shoulder__Elbow_motor">
-            <hardwareInterface>hardware_interface/PositionJointInterface</hardwareInterface>
+            <hardwareInterface>hardware_interface/VelocityJointInterface</hardwareInterface>
             <mechanicalReduction>1</mechanicalReduction>
         </actuator>
@@ -390,8 +390,8 @@
         <type>transmission_interface/SimpleTransmission</type>
         <joint name="Pitch__Roll">
-            <hardwareInterface>hardware_interface/PositionJointInterface</hardwareInterface>
+            <hardwareInterface>hardware_interface/VelocityJointInterface</hardwareInterface>
         </joint>
         <actuator name="Pitch__Roll_motor">
-            <hardwareInterface>hardware_interface/PositionJointInterface</hardwareInterface>
+            <hardwareInterface>hardware_interface/VelocityJointInterface</hardwareInterface>
             <mechanicalReduction>1</mechanicalReduction>
         </actuator>

File: prochesta_arm/urdf/prochesta_arm.urdf[backup].xacro (robot description, xacro)
@@ -26,21 +26,28 @@
         <color rgba="0.0 1.0 0.5 1.0" />
     </material>
-    <link name="base_bar">
-        <!--inertial>
+    <!-- _________________________________ -->
+    <link name="world"/>
+    <joint name="fixed_world" type="fixed">
+        <origin xyz="0.0 0.0 0.0" rpy="0.0 0.0 0.0"/>
+        <parent link="world"/>
+        <child link="base_plane"/>
+    </joint>
+    <link name="base_plane">
+        <inertial>
             <origin rpy="0 0 0" xyz="0 0 0" />
             <mass value="0.392347184025621" />
             <inertia ixx="0.0" ixy="0" ixz="0" iyy="0" iyz="0" izz="0" />
-        </inertial-->
-        <visual>
-            <origin xyz="0.0 0.0 0.05" rpy="0.0 0.0 0.0"/>
-            <geometry>
-                <box size="0.01 0.01 0.1"/>
+        </inertial>
+        <visual name="">
+            <origin xyz="0.0 0.0 0.01" rpy="0.0 0.0 0.0"/>
+            <geometry>
+                <box size="1.5 1.5 0.02"/>
             </geometry>
             <material name="grey"/>
         </visual>
         <collision>
-            <origin xyz="0.0 0.0 0.05" rpy="0.0 0.0 0.0"/>
-            <geometry>
-                <box size="0.01 0.01 0.1"/>
+            <origin xyz="0.0 0.0 0.01" rpy="0.0 0.0 0.0"/>
+            <geometry>
+                <box size="1.5 1.5 0.02"/>
             </geometry>
         </collision>
@@ -58,26 +65,27 @@
         <child link="base_bar"/>
         <axis xyz="0.0 0.0 0.0"/>
-        <limit lower="0.0" upper="0.0" effort="0.0" velocity="0.0"/>
-    </joint>
-    <link name="base_plane">
-        <!--inertial>
+        <limit lower="0.0" upper="0.0" effort="1000.0" velocity="50.0"/>
+    </joint>
+    <link name="base_bar">
+        <inertial>
             <origin rpy="0 0 0" xyz="0 0 0" />
             <mass value="0.392347184025621" />
             <inertia ixx="0.0" ixy="0" ixz="0" iyy="0" iyz="0" izz="0" />
-        </inertial-->
-        <visual name="">
-            <origin xyz="0.0 0.0 0.01" rpy="0.0 0.0 0.0"/>
-            <geometry>
-                <box size="1.5 1.5 0.02"/>
+        </inertial>
+        <visual>
+            <origin xyz="0.0 0.0 0.05" rpy="0.0 0.0 0.0"/>
+            <geometry>
+                <box size="0.01 0.01 0.1"/>
             </geometry>
             <material name="grey"/>
         </visual>
         <collision>
-            <origin xyz="0.0 0.0 0.01" rpy="0.0 0.0 0.0"/>
-            <geometry>
-                <box size="1.5 1.5 0.02"/>
-            </geometry>
-        </collision>
-    </link>
+            <origin xyz="0.0 0.0 0.05" rpy="0.0 0.0 0.0"/>
+            <geometry>
+                <box size="0.01 0.01 0.1"/>
+            </geometry>
+        </collision>
+    </link>
+    <!-- _________________________________ -->
     <link name="ArmBase">
         <inertial>
@@ -405,24 +413,4 @@
         </joint>
         <actuator name="Joint_RightClaw_motor">
-            <hardwareInterface>hardware_interface/PositionJointInterface</hardwareInterface>
-            <mechanicalReduction>1</mechanicalReduction>
-        </actuator>
-    </transmission>
-    <transmission name="trans_base_plane__ArmBase">
-        <type>transmission_interface/SimpleTransmission</type>
-        <joint name="base_plane__ArmBase">
-            <hardwareInterface>hardware_interface/PositionJointInterface</hardwareInterface>
-        </joint>
-        <actuator name="base_plane__ArmBase_motor">
-            <hardwareInterface>hardware_interface/PositionJointInterface</hardwareInterface>
-            <mechanicalReduction>1</mechanicalReduction>
-        </actuator>
-    </transmission>
-    <transmission name="trans_base_bar__base_plane">
-        <type>transmission_interface/SimpleTransmission</type>
-        <joint name="base_bar__base_plane">
-            <hardwareInterface>hardware_interface/PositionJointInterface</hardwareInterface>
-        </joint>
-        <actuator name="base_bar__base_plane_motor">
             <hardwareInterface>hardware_interface/PositionJointInterface</hardwareInterface>
             <mechanicalReduction>1</mechanicalReduction>
